File: hardware/nrf52840_addon/nrf52840_addon/esp32.kicad_sch (KiCad schematic)
At the start: 11 parts

Commit message: nrf52840_addon schematic v1
nrf52840_addon schematic v1
Parts:
- added C3, C4: 22p, symbol Device:C
- added C5, C6, C7: 0.1u, symbol Device:C
- added J10: IO_PINS_1, symbol Connector:Conn_01x04_Male
- added J11: ADC_IN, symbol Connector:Conn_01x03_Male
- added J12: IO_PINS_2, symbol Connector:Conn_01x04_Male
- added J13: ADC_IN_SEL, symbol Connector:Conn_01x03_Male
- added J14: ADC_V_SEL, symbol Connector:Conn_01x03_Male
- added J8: USB_B_Micro, symbol Connector:USB_B_Micro
- added Q1, Q2: S8050, Package_TO_SOT_THT:TO-92_Inline, symbol Transistor_BJT:S8050
- added R15, R16, R17, R18: 12K, symbol Device:R
- added R23: 5K, symbol Device:R
- added R24, R30, R32: 1K, symbol Device:R
- added R25, R31, R33: 2K, symbol Device:R
- added U11: CH340G, Package_SO:SOIC-16_3.9x9.9mm_P1.27mm, symbol Interface_USB:CH340G
- added Y1: Crystal, symbol Device:Crystal
- gave numbers to parts that had none: 11
Connections:
- net +3.3V: now also J10.1 (Pin_1), J14.3 (Pin_3), R23.1
- net GND: now also C3.2, C4.2, C5.1, C6.1, C7.2, J10.4 (Pin_4), J11.3 (Pin_3), J12.4 (Pin_4), J8.5 (GND), J8.6 (Shield), R25.2, R31.2, R33.2, U11.1 (GND)
- net DTR: now reaches U12.25 (IO0)
- net DTR: now also Q2.1 (E), R17.2, R23.2
- net RTS: now reaches C8.1, R22.2, U12.3 (EN)
- net RTS: now also Q1.3 (C), R18.2
- net PRG_RX: now reaches U12.34 (RXD0/IO3)
- net PRG_RX: now also U11.2 (TXD)
- net PRG_TX: now reaches U12.35 (TXD0/IO1)
- net PRG_TX: now also U11.3 (RXD)
- net IO_02 renamed E_LED_R
- net IO_04 renamed E_LED_G
- net IO_13 renamed E_LED_B
- net IO_34 renamed E_SW_1
- net IO_35 renamed E_SW_2
- new net: Q2.2 (B), R16.2
- new net: C5.2, U11.4 (V3)
- new net: Q1.2 (B), R15.2
- new net: C3.1, U11.7 (XI), Y1.1
- new net: C4.1, U11.8 (XO), Y1.2
- new net +5V: C6.2, C7.1, J12.1 (Pin_1), J14.1 (Pin_1), J8.1 (VBUS), U11.16 (VCC)
- new net ADC_IN_5V: J13.3 (Pin_3), R24.1
- new net ADC_IN_SEL: J11.2 (Pin_2), J13.2 (Pin_2)
- new net ADC_OUT1: J13.1 (Pin_1), R24.2, R25.1
- new net ADC_VCC: J11.1 (Pin_1), J14.2 (Pin_2)
- new net D+: J8.3 (D+), U11.5 (UD+)
- new net D-: J8.2 (D-), U11.6 (UD-)
- new net IO_IN_1: J12.2 (Pin_2), R32.1
- new net IO_IN_2: J12.3 (Pin_3), R30.1
- new net P_DTR: Q2.3 (C), R15.1, R17.1, U11.13 (~{DTR})
- new net P_RTS: Q1.1 (E), R16.1, R18.1, U11.14 (~{RTS})
- new net SPARE_1: J10.3 (Pin_3)
- new net SPARE_2: J10.2 (Pin_2)
- new net SPARE_3: R30.2, R31.1
- new net SPARE_4: R32.2, R33.1
- no-connect marks 8 -> 26
Other:
- note added: "ADC outside interface"
- note added: "ESP32 USB Programmer"
- note added: "IO interface"
- moved on the sheet: C8, D2, R13, R14, R19, R20, R21, R22, SW2, SW3, U12
