File: hardware/nrf52840_addon/nrf52840_addon/nrf52840_addon.kicad_sch (KiCad schematic)
At the start: 25 parts

Commit message: nrf52840_addon schematic v1
nrf52840_addon schematic v1
Parts:
- added J2: UART_0_PINS, symbol Connector:Conn_01x04_Male
- added J4: RX_SEL, symbol Connector:Conn_01x03_Male
- added J5: UART_V_SEL, symbol Connector:Conn_01x03_Male
- added J6: I2C connector, symbol Connector:Conn_01x04_Male
- added J7: I2C_V_SEL, symbol Connector:Conn_01x03_Male
- added J9: Ethernetpins, symbol Connector:Conn_01x08_Male
- added R2, R4: 1K, symbol Device:R
- added R3: R, symbol Device:R
- added R6: 2K, symbol Device:R
- gave numbers to parts that had none: 25
Connections:
- net 3.3V is gone; now on net +3.3V: R1.2, U2.49 (P0.09), U5.8 (LED)
- net P0_03 is gone; now on net ADC_POT: RV1.2
- net P0_04 is gone; now on net SDCARD_CS: J3.2 (DAT3/CD)
- net P0_28 is gone; now on net ADC_LM35: U9.2 (Vout)
- net +3.3V: now also J5.3 (Pin_3), J7.3 (Pin_3), J9.7 (Pin_7)
- net +5V: now also J5.1 (Pin_1), J7.1 (Pin_1)
- net GND: now also J2.4 (Pin_4), J6.2 (Pin_2), J9.8 (Pin_8), R3.2, R6.2
- net I2C0_SCL: now also J6.4 (Pin_4)
- net I2C0_SDA: now also J6.3 (Pin_3)
- net P1_05: no longer SW1.B, U2.43 (P1.05)
- net SPI1_MISO: now also J9.3 (Pin_3); no longer J3.7 (DAT0)
- net SPI1_MOSI: now also J9.2 (Pin_2); no longer J3.3 (CMD)
- net SPI1_SCK: now also J9.1 (Pin_1); no longer J3.5 (CLK)
- net SPI2-QSPI-IO0: now also J3.7 (DAT0)
- net SPI2-QSPI-IO1: now also J3.3 (CMD)
- net SPI2-QSPI-IO2: now also J3.8 (DAT1)
- net SPI2-QSPI-IO3: now also J3.1 (DAT2)
- net SPI2-QSPI-SCK: now also J3.5 (CLK)
- net UART0_RX: now also J4.1 (Pin_1), R2.2, R3.1
- net UART0_TX: now also J2.1 (Pin_1)
- net BTN_0: no longer names the net of U2.21 (P0.11)
- net BTN_1: no longer names the net of U2.56 (P0.12)
- net BTN_2: no longer names the net of U2.62 (P0.24)
- net BTN_3: no longer names the net of U2.28 (P0.25)
- net DETECT: no longer names the net of U2.20 (DETECT)
- net LED_0: no longer names the net of U2.22 (P0.13)
- net LED_1: no longer names the net of U2.57 (P0.14)
- net LED_2: no longer names the net of U2.23 (P0.15)
- net LED_3: no longer names the net of U2.58 (P0.16)
- net MX25R6435F_CS: no longer names the net of U2.24 (P0.17)
- net P0_00 renamed NEOPIXEL
- net P0_01 renamed SPARE_3
- net P0_02 renamed ETH_RESET
- net ETH_RESET: now also J9.5 (Pin_5)
- net P0_05 renamed DIS_CS
- net P0_07 renamed DHT22
- net P0_10 renamed DIS_A0
- net P0_18 renamed SPARE_4
- net P0_29 renamed ADC_OUT1
- net P1_00 renamed SPARE_1
- net P1_03 renamed ENCODE_A
- net P1_04 renamed ENCODE_B
- net P1_06 renamed ETH_CS
- net ETH_CS: now also J9.4 (Pin_4)
- net P1_07 renamed SPARE_2
- net P1_09 renamed ETH_INT
- net ETH_INT: now also J9.6 (Pin_6)
- net P1_10: no longer names the net of J1.2 (Pin_2)
- net P1_10: now also R4.2; no longer U2.39 (P1.10)
- net P1_11 renamed US_TRIG
- net P1_12 renamed LED_R
- net P1_13 renamed LED_G
- net LED_G: no longer U2.19 (P1.13)
- net P1_14 renamed LED_B
- net LED_B: no longer U2.15 (P1.14)
- net P1_15 renamed DS18B20
- net DS18B20: no longer U2.16 (P1.15)
- new net ENCODE_C: SW1.B, U2.43 (P1.05)
- new net I2C_VCC: J6.1 (Pin_1), J7.2 (Pin_2)
- new net UART0_RX_5V: J4.3 (Pin_3), R2.1
- new net UART0_RX_SEL: J2.2 (Pin_2), J4.2 (Pin_2)
- new net UART_VCC: J2.3 (Pin_3), J5.2 (Pin_2)
- new net US_ECHO: R4.1, R6.1, U2.39 (P1.10)
- no-connect marks 12 -> 24
Other:
- note added: "DHT22 interface"
- note added: "DS18B20 interface"
- note added: "LM35 interface"
- note added: "RGB led interface"
- note added: "SDcard interface"
- note added: "SPI Display interface"
- note added: "UART0 interface"
- note added: "Ultrasonic interface"
- note added: "WS2812B neopixel interface"
- note added: "encoder interface"
- note added: "ethernet interface"
- note added: "potentiometer"
- note removed: "WS2812B"
- moved on the sheet: C2, D1, J1, R1, R10, R11, R12, R5, R7, R8, R9, RV1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
